Commit message: Split Primuus thigh collision meshes to avoid hull overlap

File: src/controller/rl/resources/robots/primuus/urdf/primuus.urdf (robot description, URDF)
Before this commit: robot primuus, 17 links, 16 joints
Links:
- link FL_thigh_link: geometry collision mesh filename=../collision/FL_thigh_motor.STL; collision mesh filename=../collision/FL_thigh_plate.STL
- link FR_thigh_link: geometry collision mesh filename=../collision/FR_thigh_motor.STL; collision mesh filename=../collision/FR_thigh_plate.STL
- link RL_thigh_link: geometry collision mesh filename=../collision/RL_thigh_motor.STL; collision mesh filename=../collision/RL_thigh_plate.STL
- link RR_thigh_link: geometry collision mesh filename=../collision/RR_thigh_motor.STL; collision mesh filename=../collision/RR_thigh_plate.STL

Commit message: Add Primuus MuJoCo model and deployment config

File: src/controller/rl/resources/robots/primuus/urdf/primuus.urdf (robot description, URDF)
Before this commit: robot primuus, 17 links, 16 joints
Joints:
- joint FL_calf_joint: limit lower=-2.7227 upper=-0.8378 effort=45.43 velocity=15.7 -> lower=-2.7227 upper=-0.8378 effort=23.7 velocity=15.7
- joint FR_calf_joint: limit lower=-2.7227 upper=-0.8378 effort=45.43 velocity=15.7 -> lower=-2.7227 upper=-0.8378 effort=23.7 velocity=15.7
- joint RL_calf_joint: limit lower=-2.7227 upper=-0.8378 effort=45.43 velocity=15.7 -> lower=-2.7227 upper=-0.8378 effort=23.7 velocity=15.7
- joint RR_calf_joint: limit lower=-2.7227 upper=-0.8378 effort=45.43 velocity=15.7 -> lower=-2.7227 upper=-0.8378 effort=23.7 velocity=15.7

Commit message: Align Primuus collision geometry and safe joint workspace

File: src/controller/rl/resources/robots/primuus/urdf/primuus.urdf (robot description, URDF)
Before this commit: robot primuus, 17 links, 16 joints
Links:
- link FL_calf_link: geometry collision mesh filename=../collision/convex/FL_calf_main.obj; visual mesh filename=../stl/FL_calf_link.STL
- link FL_thigh_link: geometry collision mesh filename=../collision/FL_thigh_motor.STL; collision mesh filename=../collision/convex/FL_thigh_feature_00.obj
- link FR_calf_link: geometry collision mesh filename=../collision/convex/FR_calf_main.obj; visual mesh filename=../stl/FR_calf_link.STL
- link FR_thigh_link: geometry collision mesh filename=../collision/FR_thigh_motor.STL; collision mesh filename=../collision/convex/FR_thigh_feature_00.obj
- link RL_calf_link: geometry collision mesh filename=../collision/convex/RL_calf_main.obj; visual mesh filename=../stl/RL_calf_link.STL
- link RL_thigh_link: geometry collision mesh filename=../collision/RL_thigh_motor.STL; collision mesh filename=../collision/convex/RL_thigh_feature_00.obj
- link RR_calf_link: geometry collision mesh filename=../collision/convex/RR_calf_main.obj; visual mesh filename=../stl/RR_calf_link.STL
- link RR_thigh_link: geometry collision mesh filename=../collision/RR_thigh_motor.STL; collision mesh filename=../collision/convex/RR_thigh_feature_00.obj
Joints:
- joint FL_calf_joint: limit lower=-2.7227 upper=-0.8378 effort=23.7 velocity=15.7 -> lower=-2.4 upper=-0.8378 effort=23.7 velocity=15.7
- joint FR_calf_joint: limit lower=-2.7227 upper=-0.8378 effort=23.7 velocity=15.7 -> lower=-2.4 upper=-0.8378 effort=23.7 velocity=15.7
- joint RL_calf_joint: limit lower=-2.7227 upper=-0.8378 effort=23.7 velocity=15.7 -> lower=-2.4 upper=-0.8378 effort=23.7 velocity=15.7
- joint RR_calf_joint: limit lower=-2.7227 upper=-0.8378 effort=23.7 velocity=15.7 -> lower=-2.4 upper=-0.8378 effort=23.7 velocity=15.7

Commit message: Restore Primuus joint range and enable calf self-collisions

File: src/controller/rl/resources/robots/primuus/urdf/primuus.urdf (robot description, URDF)
Before this commit: robot primuus, 17 links, 16 joints
Links:
- added link FL_calf_collision_link, mass 0.069695803833827993; collision mesh filename=../collision/convex/FL_calf_part_00.obj; collision mesh filename=../collision/convex/FL_calf_part_01.obj
- added link FR_calf_collision_link, mass 0.069695803833827993; collision mesh filename=../collision/convex/FR_calf_part_00.obj; collision mesh filename=../collision/convex/FR_calf_part_01.obj
- added link RL_calf_collision_link, mass 0.069695803833821499; collision mesh filename=../collision/convex/RL_calf_part_00.obj; collision mesh filename=../collision/convex/RL_calf_part_01.obj
- added link RR_calf_collision_link, mass 0.069695803833825495; collision mesh filename=../collision/convex/RR_calf_part_00.obj; collision mesh filename=../collision/convex/RR_calf_part_01.obj
- link FL_calf_link: mass 0.139391607667656 -> 0.069695803833827993; geometry visual mesh filename=../stl/FL_calf_link.STL
- link FR_calf_link: mass 0.139391607667656 -> 0.069695803833827993; geometry visual mesh filename=../stl/FR_calf_link.STL
- link RL_calf_link: mass 0.139391607667643 -> 0.069695803833821499; geometry visual mesh filename=../stl/RL_calf_link.STL
- link RR_calf_link: mass 0.139391607667651 -> 0.069695803833825495; geometry visual mesh filename=../stl/RR_calf_link.STL
Joints:
- added joint FL_calf_collision_joint: type fixed, parent FL_calf_link, child FL_calf_collision_link, origin xyz=0 0 0 rpy=0 0 0
- added joint FR_calf_collision_joint: type fixed, parent FR_calf_link, child FR_calf_collision_link, origin xyz=0 0 0 rpy=0 0 0
- added joint RL_calf_collision_joint: type fixed, parent RL_calf_link, child RL_calf_collision_link, origin xyz=0 0 0 rpy=0 0 0
- added joint RR_calf_collision_joint: type fixed, parent RR_calf_link, child RR_calf_collision_link, origin xyz=0 0 0 rpy=0 0 0
- joint FL_calf_joint: limit lower=-2.4 upper=-0.8378 effort=23.7 velocity=15.7 -> lower=-2.7227 upper=-0.8378 effort=23.7 velocity=15.7
- joint FR_calf_joint: limit lower=-2.4 upper=-0.8378 effort=23.7 velocity=15.7 -> lower=-2.7227 upper=-0.8378 effort=23.7 velocity=15.7
- joint RL_calf_joint: limit lower=-2.4 upper=-0.8378 effort=23.7 velocity=15.7 -> lower=-2.7227 upper=-0.8378 effort=23.7 velocity=15.7
- joint RR_calf_joint: limit lower=-2.4 upper=-0.8378 effort=23.7 velocity=15.7 -> lower=-2.7227 upper=-0.8378 effort=23.7 velocity=15.7
