Commit message: Sync simplified Primuus collision assets and document local regression

File: resources/robots/primuus/urdf/primuus.urdf (robot description, URDF)
Before this commit: robot primuus, 21 links, 20 joints
Links:
- link FL_thigh_link: geometry collision mesh filename=../collision/FL_thigh_motor.STL; collision mesh filename=../collision/convex/FL_thigh_feature_00.obj
- link FR_thigh_link: geometry collision mesh filename=../collision/FR_thigh_motor.STL; collision mesh filename=../collision/convex/FR_thigh_feature_00.obj
- link RL_thigh_link: geometry collision mesh filename=../collision/RL_thigh_motor.STL; collision mesh filename=../collision/convex/RL_thigh_feature_00.obj
- link RR_thigh_link: geometry collision mesh filename=../collision/RR_thigh_motor.STL; collision mesh filename=../collision/convex/RR_thigh_feature_00.obj

Commit message: Restore original Primuus clearance meshes and sync equivalent body hulls

File: resources/robots/primuus/urdf/primuus.urdf (robot description, URDF)
Before this commit: robot primuus, 21 links, 20 joints
Links:
- link FL_hip_link: geometry collision mesh filename=../collision/convex/FL_hip_link_collision_hull.obj; visual mesh filename=../stl/FL_hip_link.STL
- link FL_thigh_link: geometry collision mesh filename=../collision/FL_thigh_motor.STL; collision mesh filename=../collision/convex/FL_thigh_feature_00.obj
- link FR_hip_link: geometry collision mesh filename=../collision/convex/FR_hip_link_collision_hull.obj; visual mesh filename=../stl/FR_hip_link.STL
- link FR_thigh_link: geometry collision mesh filename=../collision/FR_thigh_motor.STL; collision mesh filename=../collision/convex/FR_thigh_feature_00.obj
- link RL_hip_link: geometry collision mesh filename=../collision/convex/RL_hip_link_collision_hull.obj; visual mesh filename=../stl/RL_hip_link.STL
- link RL_thigh_link: geometry collision mesh filename=../collision/RL_thigh_motor.STL; collision mesh filename=../collision/convex/RL_thigh_feature_00.obj
- link RR_hip_link: geometry collision mesh filename=../collision/convex/RR_hip_link_collision_hull.obj; visual mesh filename=../stl/RR_hip_link.STL
- link RR_thigh_link: geometry collision mesh filename=../collision/RR_thigh_motor.STL; collision mesh filename=../collision/convex/RR_thigh_feature_00.obj
- link base_link: geometry collision mesh filename=../collision/convex/base_link_collision_hull.obj; visual mesh filename=../stl/base_link.STL

Commit message: Sync 65-shape Primuus collision assets and preserve cylinder geometry

File: resources/robots/primuus/urdf/primuus.urdf (robot description, URDF)
Before this commit: robot primuus, 21 links, 20 joints
Links:
- link FL_thigh_link: geometry collision box size=0.003 0.025 0.047887889909663; collision cylinder length=0.025 radius=0.04
- link FR_thigh_link: geometry collision box size=0.003 0.025 0.047887889909663; collision cylinder length=0.025 radius=0.04
- link RL_thigh_link: geometry collision box size=0.003 0.025 0.047887889909663; collision cylinder length=0.025 radius=0.04
- link RR_thigh_link: geometry collision box size=0.003 0.025 0.047887889909663; collision cylinder length=0.025 radius=0.04

Commit message: Align Primuus thigh offset and record local-only contact screening

File: resources/robots/primuus/urdf/primuus.urdf (robot description, URDF)
Before this commit: robot primuus, 21 links, 20 joints
Joints:
- joint RL_thigh_joint: origin xyz=-0.082063 0.0346 0 rpy=0 0 0 -> xyz=-0.082063 0.0343 0 rpy=0 0 0
